File: merged/IR-endstop.sch (KiCad schematic (older format))
At the start: 8 parts, among them P1 CONN_01X03, Q1 2N7002KT1G, U1 EE-SX1103

Commit message: rev.041
Parts:
- D2: symbol IR-endstop-04-rescue:D_ALT-device-DLP-control-rescue-DLP-control-04-rescue-DLP-control-05-rescue-SL1-control-05b-rescue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 -> IR-endstop-0.4.1-rescue:D_ALT-device-DLP-control-rescue-DLP-control-04-rescue-DLP-control-05-rescue-SL1-control-05b-res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
- P1: symbol conn:CONN_01X03 -> IR-endstop-0.4.1-rescue:CONN_01X03-conn
- Q1: symbol transistors:2N7002 -> IR-endstop-0.4.1-rescue:2N7002-transistors
- R1, R2, R3, R4: symbol device:R -> IR-endstop-0.4.1-rescue:R-device
- U1: symbol opto:LTV-817 -> IR-endstop-0.4.1-rescue:LTV-817-opto
Other:
- note added: "Changelog\n--------\nrev 0.4.1\n- modify footprints\nrev 0.4\n= 0.3b s with new silkscreen\nrev 0.3b\n- add R4\nrev 0.3\n- add D2"
- note removed: "Changelog\n--------\nrev 0.4\n- add R4\nrev 0.3\n- add D2"
Changed lines of the file:
@@
 Sheet 1 1
 Title "IR sensor"
-Date "2019-07-04"
-Rev "0.4"
-Comp "Prusa Development a.s."
+Date "2020-06-24"
+Rev "0.4.1"
+Comp "PRUSA RESEARCH s.r.o"
 Comment1 "http://creativecommons.org/licenses/by-sa/4.0/"
 Comment2 "Licensed under the Attribution-ShareAlike 4.0 International (CC BY-SA 4.0)"
@@
 $EndDescr
 $Comp
-L opto:LTV-817 U1
+L IR-endstop-0.4.1-rescue:LTV-817-opto U1
 U 1 1 5BD7084A
 P 4950 3975
@@
 $EndComp
 $Comp
-L conn:CONN_01X03 P1
+L IR-endstop-0.4.1-rescue:CONN_01X03-conn P1
 U 1 1 5BD70990
 P 7525 3575
@@
 $EndComp
 $Comp
-L device:R R1
+L IR-endstop-0.4.1-rescue:R-device R1
 U 1 1 5BD709E3
 P 4500 3875
@@
 +5V\nOUT\nGND
 $Comp
-L device:R R2
+L IR-endstop-0.4.1-rescue:R-device R2
 U 1 1 5BD6C176
 P 5400 3675
@@
 	6025 3575 6025 3625
 $Comp
-L device:R R3
+L IR-endstop-0.4.1-rescue:R-device R3
 U 1 1 5BE2C39F
 P 5750 3575
@@
 0,32V
 $Comp
-L transistors:2N7002 Q1
+L IR-endstop-0.4.1-rescue:2N7002-transistors Q1
 U 1 1 5BE32902
 P 5925 3825
@@
 	7050 3875 7050 3675
 $Comp
-L IR-endstop-04-rescue:D_ALT-device-DLP-control-rescue-DLP-control-04-rescue-DLP-control-05-rescue-SL1-control-05b-rescue-SL-controller-06-rescue-SL-controller-06b-rescue-SL-controller-06c-rescue-IR-endstop-03-rescue-IR-endstop-03b-rescue D2
+L IR-endstop-0.4.1-rescue:D_ALT-device-DLP-control-rescue-DLP-control-04-rescue-DLP-control-05-rescue-SL1-control-05b-rescue-SL-controller-06-rescue-SL-controller-06b-rescue-SL-controller-06c-rescue-IR-endstop-03-rescue-IR-endstop-03b-rescue-IR-endstop-04-rescue D2
 U 1 1 5D0C3FD7
 P 7050 4025
@@
 GND
 Text Notes 6100 7450 0    50   ~ 0
-Changelog\n--------\nrev 0.4\n- add R4\nrev 0.3\n- add D2
+Changelog\n--------\nrev 0.4.1\n- modify footprints\nrev 0.4\n= 0.3b s with new silkscreen\nrev 0.3b\n- add R4\nrev 0.3\n- add D2
 $Comp
-L device:R R4
+L IR-endstop-0.4.1-rescue:R-device R4
 U 1 1 5D1DA941
 P 6800 3675
